File: mp3.kicad_pcb (KiCad board)
At the start: 2 copper layers, 35 x 75 mm, 33 parts, among them J1 Conn_02x04_Odd_Even, J2 24V in, J3 Analog power, J4 2.5mm Jack, J5 Micro_SD_Card, SW1 SW_SPDT, U1 LM2596S-3.3, U2 STM32G431K8T6, U3 LD1086DT33TR, U4 PCM5102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

Commit message: v0.2
Parts:
- removed J1: Conn_02x04_Odd_Even, Connector_PinHeader_2.54mm:PinHeader_2x04_P2.54mm_Vertical
- added C17: C, Capacitor_SMD:C_0805_2012Metric, F.Cu at (137.9, 96.2)
- added C18: C, Capacitor_SMD:C_0805_2012Metric, F.Cu at (142.1, 96.2)
- added C19: 10u, Capacitor_SMD:C_0805_2012Metric, F.Cu at (144.1, 96.2)
- added D1: 40V, Diode_SMD:D_SOD-123F, F.Cu at (156.1, 58.2)
- added J6: RJ45_Bel_SI-60062-F, Connector_RJ:RJ45_Bel_SI-60062-F, F.Cu at (143.4, 64.5)
- added R4: R, Resistor_SMD:R_0805_2012Metric, F.Cu at (139.9, 96.2)
- added R5: 470R, Resistor_SMD:R_0805_2012Metric, F.Cu at (135.9, 96.2)
- added R6: 470R, Resistor_SMD:R_0805_2012Metric, F.Cu at (133.9, 96.2)
- added TP1: TestPoint, TestPoint:TestPoint_Pad_D1.0mm, F.Cu at (157.6, 105.1)
- added TP10: TestPoint, TestPoint:TestPoint_Pad_D1.0mm, F.Cu at (170.7, 101.9)
- added TP11: TestPoint, TestPoint:TestPoint_Pad_D1.0mm, F.Cu at (173.7, 108.8)
- added TP12: TestPoint, TestPoint:TestPoint_Pad_D1.0mm, F.Cu at (170.6, 80.0)
- added TP2: TestPoint, TestPoint:TestPoint_Pad_D1.0mm, F.Cu at (151.5, 106.0)
- added TP3: TestPoint, TestPoint:TestPoint_Pad_D1.0mm, F.Cu at (154.0, 106.0)
- added TP4: TestPoint, TestPoint:TestPoint_Pad_D1.0mm, F.Cu at (166.0, 89.8)
- added TP6: TestPoint, TestPoint:TestPoint_Pad_D1.0mm, F.Cu at (157.5, 102.2)
- added TP7: TestPoint, TestPoint:TestPoint_Pad_D1.0mm, F.Cu at (166.0, 91.9)
- added TP8: TestPoint, TestPoint:TestPoint_Pad_D1.0mm, F.Cu at (171.2, 99.1)
- added TP9: TestPoint, TestPoint:TestPoint_Pad_D1.0mm, F.Cu at (166.0, 94.0)
- added U5: ENC28J60x-SS, Package_SO:SSOP-28_5.3x10.2mm_P0.65mm, F.Cu at (141.2, 85.9)
- added Y2: 25MHz, Crystal:Crystal_HC49-4H_Vertical, F.Cu at (141.4, 100.8)
- C11, C12, C7: footprint Capacitor_SMD:C_0805_2012Metric -> Capacitor_SMD:C_0603_1608Metric
- C6: footprint Capacitor_SMD:C_1206_3216Metric -> Capacitor_SMD:C_0805_2012Metric
- moved H1 18.0 mm to (134.0, 52.0)
- moved L1 1.10 mm to (164.2, 54.5)
- moved H2 1.00 mm to (178.0, 117.0)
- moved C14 0.11 mm to (180.5, 97.9)
- moved C1 0.10 mm to (155.4, 96.5)
- moved C2 0.10 mm to (157.6, 96.5)
- moved R1 0.06 mm to (155.5, 100.1)
Connections:
- J5 pad 1: (no net) -> no_connect_45
- J5 pad 8: (no net) -> no_connect_46
- U2 pad 20: (no net) -> no_connect_49
- U2 pad 21: (no net) -> no_connect_50
- U2 pad 22: (no net) -> no_connect_51
- U2 pad 23: (no net) -> no_connect_52
- U2 pad 24: (no net) -> no_connect_53
- U2 pad 27: (no net) -> no_connect_54
- U2 pad 29: (no net) -> no_connect_55
- U2 pad 30: (no net) -> no_connect_56
- U2 pad 31: BOOT0 -> Net-(U2-Pad31)
- U2 pad 4: Recet -> Net-(U2-Pad4)
- U2 pad 5: (no net) -> no_connect_57
- U2 pad 6: (no net) -> no_connect_58
- U2 pad 7: (no net) -> SPI_ETH_CS
- U2 pad 8: (no net) -> no_connect_59
- U2 pad 9: (no net) -> no_connect_60
Routing:
- net +3V3: track 192.2 -> 231.0 mm, vias 5 -> 9
- net Net-(J6-PadL1): track 0.00 -> 36.7 mm
- net SPI_CLK: track 21.0 -> 53.2 mm
- net SPI_ETH_CS: track 0.00 -> 30.4 mm
- net Net-(J6-PadL3): track 0.00 -> 27.8 mm
- net SPI_MISO: track 26.0 -> 52.7 mm
- net SPI_MOSI: track 28.4 -> 52.6 mm, vias 1 -> 2
- net /ETH_T+: track 0.00 -> 24.1 mm, vias 0 -> 2
- net /ETH_T-: track 0.00 -> 19.4 mm
- net GND: track 59.4 -> 41.5 mm, vias 35 -> 47
- net BOOT0: track 17.6 -> 0.00 mm, vias 1 -> 0
- net /ETH_R+: track 0.00 -> 17.1 mm
- net /ETH_OSC1: track 0.00 -> 16.6 mm
- net /ETH_R-: track 0.00 -> 14.6 mm
- net /ETH_OSC2: track 0.00 -> 9.29 mm
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Other:
- board size 35 x 75 mm -> 54 x 75 mm
- board text added: "3,5 mm audio jack Center hight: 4.3 mm"
- board text added: "ETH PHY"
- board text added: "Ehternet"
- board text added: "TP1 SPI_CLK (25.4, 16.9)"
- board text added: "TP10 I2S_ (12.3, 20.1)"
- board text added: "TP11 I2S_SYS_CLK (9.3, 13.2)"
- board text added: "TP2 SPI_MISO (31.5, 16)"
- board text added: "TP3 SPI_MOSI (29, 16)"
- board text added: "TP4 +3.3VA (12.4, 42)"
- board text added: "TP4 +3.3VD (17, 32.2)"
- board text added: "TP6 BOOT0 (25.5, 19.8)"
- board text added: "TP7 BOOT0 (17, 30.1)"
- board text added: "TP8 I2S_LR_CLK (11, 22.9)"
- board text added: "TP9 I2C_(SD) (17, 30.1)"
- board text added: "micro SD Card"
- board text added: "of/off switch (^: on; v: off) hieght: ??"
