File: mp3.kicad_sch (KiCad schematic)
At the start: 34 parts, among them J1 Conn_02x04_Odd_Even, J2 24V in, J3 Analog power, J4 2.5mm Jack, J5 Micro_SD_Card, SW1 SW_SPDT, U1 LM2596S-3.3, U2 STM32G431K8T6, U3 LD1086DT33TR, U4 PCM5102, Y1 8MHz

Commit message: v0.2
Parts:
- removed J1: Conn_02x04_Odd_Even, Connector_PinHeader_2.54mm:PinHeader_2x04_P2.54mm_Vertical, symbol Connector_Generic:Conn_02x04_Odd_Even
- added C17, C18: C, Capacitor_SMD:C_0805_2012Metric, symbol Device:C
- added C19: 10u, Capacitor_SMD:C_0805_2012Metric, symbol Device:C
- added J6: RJ45_Bel_SI-60062-F, Connector_RJ:RJ45_Bel_SI-60062-F, symbol Connector:RJ45_Bel_SI-60062-F
- added R4: R, Resistor_SMD:R_0805_2012Metric, symbol Device:R
- added R5, R6: 470R, Resistor_SMD:R_0805_2012Metric, symbol Device:R
- added TP1, TP10, TP11, TP12, TP2, TP3, TP4, TP6, TP7, TP8, TP9: TestPoint, TestPoint:TestPoint_Pad_D1.0mm, symbol Connector:TestPoint
- added U5: ENC28J60x-SS, Package_SO:SSOP-28_5.3x10.2mm_P0.65mm, symbol Interface_Ethernet:ENC28J60x-SS
- added Y2: 25MHz, Crystal:Crystal_HC49-4H_Vertical, symbol Device:Crystal
- D1: footprint (none) -> Diode_SMD:D_SOD-123F
Connections:
- net +3.3VA: now also TP12.1
- net +3V3: now also TP4.1, U5.15 (VDDTX), U5.19 (VDDRX), U5.20 (VDDPLL), U5.25 (VDDOSC), U5.28 (VDD)
- net GND: now also C17.1, C18.1, C19.2, J6.8 (GND), J6.L2 (LEDY_K), J6.L4 (LEDG_K), J6.SH (SHIELD), U5.10 (~RESET), U5.11 (VSSRX), U5.18 (VSSTX), U5.2 (VSS), U5.21 (VSSPLL), U5.22 (VSSOSC)
- net I2S3_BCK: now also TP10.1
- net I2S3_LRCK: now also TP8.1
- net I2S3_SCK: now also TP11.1
- net I2S3_SD: now also TP9.1
- net SPI_CLK: now also TP1.1, U5.8 (SCK)
- net SPI_MISO: now also TP2.1, U5.6 (SO)
- net SPI_MOSI: now also TP3.1, U5.7 (SI)
- net SPI_ETH_CS: now reaches U2.7 (PA2)
- net SPI_ETH_CS: now also U5.9 (~CS)
- net BOOT0: no longer names the net of U2.31 (PB8-BOOT0)
- net BOOT0: now also TP7.1
- net Recet: no longer names the net of U2.4 (PG10-NRST)
- net Recet: now also TP6.1
- new net: J6.L3 (LEDG_A), R5.2
- new net: C17.2, R4.1, Y2.2
- new net: C19.1, U5.1 (VCAP)
- new net: J6.L1 (LEDY_A), R6.2
- new net ETH_LEDA: R5.1, U5.27 (LEDA)
- new net ETH_LEDB: R6.1, U5.26 (LEDB)
- new net ETH_OSC1: C18.2, U5.23 (OSC1), Y2.1
- new net ETH_OSC2: R4.2, U5.24 (OSC2)
- new net ETH_R+: J6.4 (RD+), U5.13 (TPIN+)
- new net ETH_R-: J6.6 (RD-), U5.12 (TPIN-)
- new net ETH_T+: J6.1 (TD+), U5.17 (TPOUT+)
- new net ETH_T-: J6.3 (TD-), U5.16 (TPOUT-)
- no-connect marks 16 -> 19
Other:
- note added: "ETH"
- note removed: "Progamming header"
- company: (none) -> MReenen
- title: (none) -> MP3 Player
- moved on the sheet: C10, C11, C12, C13, C14, C15, C16, C3, C4, C5, C6, C7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
