File: MP3 - Mats van Reenen/kicad 6 files/mp3.kicad_pcb (KiCad board)
At the start: 2 copper layers, 54 x 75 mm, 54 parts, among them J2 24V in, J3 Analog power, J4 2.5mm Jack, J5 Micro_SD_Card, J6 RJ45_Bel_SI-60062-F, SW1 SW_SPDT, U1 LM2596S-3.3, U2 STM32G431K8T6, U3 LD1086DT33TR, U4 PCM5102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

Commit message: 1.0
Other:
- board text added: "TP10 I2S_ (12.3, 20.1)"
- board text added: "TP11 I2S_SYS_CLK (9.3, 13.2)"
- board text added: "TP6 BOOT0 (25.5, 19.8)"
- board text added: "TP8 I2S_LR_CLK (11, 22.9)"
- board text added: "TP9 I2C_(SD) (17, 30.1)"
- board text removed: "Power Switch"
- board text removed: "TP10 I2S_BCK (12.3, 20.1)"
- board text removed: "TP11 I2S_SCK (9.3, 13.2)"
- board text removed: "TP6 NRST (25.5, 19.8)"
- board text removed: "TP8 I2S_LRCK (11, 22.9)"
- board text removed: "TP9 I2S_SD (17, 30.1)"
- board text removed: "audio jack"
- board text removed: "micro SD-card"
Changed lines of the file:
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@@
     (aux_axis_origin 183 122)
     (pcbplotparams
-      (layerselection 0x02410f0_ffffffff)
+      (layerselection 0x03c10f0_ffffffff)
       (disableapertmacros false)
       (usegerberextensions false)
@@
     (property "Sheet name" "")
     (attr through_hole)
-    (fp_text reference "SW1" (at -2 -4 90) (layer "F.SilkS")
+    (fp_text reference "SW1" (at 4 -3.3 90) (layer "F.SilkS")
       (effects (font (size 1 1) (thickness 0.15)))
     )
@@
     (property "Sheet name" "")
     (attr smd)
-    (fp_text reference "J5" (at 7.6 1.5) (layer "F.SilkS")
+    (fp_text reference "J5" (at 7.6 1) (layer "F.SilkS")
       (effects (font (size 1 1) (thickness 0.15)))
     )
@@
     (property "Sheet name" "")
     (attr through_hole)
-    (fp_text reference "J4" (at -5 0 180) (layer "F.SilkS")
+    (fp_text reference "J4" (at 0.1 14 90) (layer "F.SilkS")
       (effects (font (size 1 1) (thickness 0.15)))
     )
@@
     (property "Sheet name" "")
     (attr smd)
-    (fp_text reference "U3" (at 3 -4.248) (layer "F.SilkS")
+    (fp_text reference "U3" (at 5 -4.248) (layer "F.SilkS")
       (effects (font (size 1 1) (thickness 0.15)))
     )
@@
     (property "Sheet name" "")
     (attr exclude_from_pos_files)
-    (fp_text reference "TP4" (at -3 -0.3) (layer "F.SilkS")
+    (fp_text reference "TP4" (at 0 -1.5) (layer "F.SilkS")
       (effects (font (size 1 1) (thickness 0.15)))
     )
@@
     (effects (font (size 1.25 1.25) (thickness 0.2)))
   )
-  (gr_text "audio jack" (at 167 86 90) (layer "F.SilkS")
-    (effects (font (size 1 1) (thickness 0.15)))
-  )
-  (gr_text "Ehternet\n" (at 140 56.5) (layer "F.SilkS")
+  (gr_text "Ehternet\n" (at 141 57) (layer "F.SilkS")
     (effects (font (size 2 2) (thickness 0.3)))
   )
@@
     (effects (font (size 1 1) (thickness 0.15)))
   )
-  (gr_text "micro SD-card" (at 171 114) (layer "F.SilkS")
-    (effects (font (size 1 1) (thickness 0.15)))
-  )
-  (gr_text "Power Switch" (at 172.5 53.5 90) (layer "F.SilkS")
-    (effects (font (size 1 1) (thickness 0.15)))
-  )
   (gr_text "DAC" (at 179 107) (layer "F.SilkS")
     (effects (font (size 2 2) (thickness 0.3)))
@@
     (effects (font (size 1 1) (thickness 0.15)))
   )
-  (gr_text "TP8\nI2S_LRCK\n(11, 22.9)" (at 167.7 98.9) (layer "User.4")
+  (gr_text "TP8\nI2S_LR_CLK\n(11, 22.9)" (at 167.7 98.9) (layer "User.4")
     (effects (font (size 0.5 0.5) (thickness 0.08)))
   )
@@
     (effects (font (size 0.5 0.5) (thickness 0.08)))
   )
-  (gr_text "TP11\nI2S_SCK\n(9.3, 13.2)" (at 170.4 109.3) (layer "User.4")
+  (gr_text "TP11\nI2S_SYS_CLK\n(9.3, 13.2)" (at 170.4 109.3) (layer "User.4")
     (effects (font (size 0.5 0.5) (thickness 0.08)))
   )
@@
     (effects (font (size 0.5 0.5) (thickness 0.08)))
   )
-  (gr_text "TP6\nNRST\n(25.5, 19.8)" (at 155.5 99.9) (layer "User.4")
+  (gr_text "TP6\nBOOT0\n(25.5, 19.8)" (at 155.5 99.9) (layer "User.4")
     (effects (font (size 0.5 0.5) (thickness 0.08)))
   )
@@
     (effects (font (size 0.5 0.5) (thickness 0.08)))
   )
-  (gr_text "TP9\nI2S_SD\n(17, 30.1)" (at 162.3 94.5) (layer "User.4")
+  (gr_text "TP9\nI2C_(SD)\n(17, 30.1)" (at 162.3 94.5) (layer "User.4")
     (effects (font (size 0.5 0.5) (thickness 0.08)))
   )
@@
     (effects (font (size 0.5 0.5) (thickness 0.08)))
   )
-  (gr_text "TP10\nI2S_BCK\n(12.3, 20.1)" (at 168.4 102.9) (layer "User.4")
+  (gr_text "TP10\nI2S_\n(12.3, 20.1)" (at 168.4 102.9) (layer "User.4")
     (effects (font (size 0.5 0.5) (thickness 0.08)))
   )
@@
   (dimension (type orthogonal) (layer "User.2")
     (pts (xy 183 83.7) (xy 186 83.7))
-    (height 1.7)
+    (height -1.7)
     (orientation 0)
     (gr_text "3 mm" (at 185.5 80) (layer "User.2")
@@
   (dimension (type orthogonal) (layer "User.2")
     (pts (xy 183 50.2) (xy 190.2 50.2))
-    (height 4.2)
+    (height -4.2)
     (orientation 0)
     (gr_text "7 mm" (at 186.5 44) (layer "User.2")
